Commit message: wip: prep pkgs for prius_simulator

File: prius_vehicle_description/urdf/vehicle.xacro (robot description, xacro)
@@ -2,5 +2,5 @@
 <robot xmlns:xacro="http://ros.org/wiki/xacro">
   <!-- load parameter -->
-  <xacro:property name="vehicle_info" value="${xacro.load_yaml('$(find sample_vehicle_description)/config/vehicle_info.param.yaml')}"/>
+  <xacro:property name="vehicle_info" value="${xacro.load_yaml('$(find prius_vehicle_description)/config/vehicle_info.param.yaml')}"/>
   <!-- vehicle body -->
   <link name="base_link">
@@ -8,5 +8,5 @@
       <origin xyz="${vehicle_info['/**']['ros__parameters']['wheel_base']/2.0} 0 0" rpy="${pi/2.0} 0 ${pi}"/>
       <geometry>
-        <mesh filename="package://sample_vehicle_description/mesh/lexus.dae" scale="1 1 1"/>
+        <mesh filename="package://prius_vehicle_description/mesh/lexus.dae" scale="1 1 1"/>
       </geometry>
     </visual>

Commit message: wip: for prius sim

File: prius_vehicle_description/urdf/vehicle.xacro (robot description, xacro)
@@ -2,13 +2,13 @@
 <robot xmlns:xacro="http://ros.org/wiki/xacro">
   <!-- load parameter -->
-  <xacro:property name="vehicle_info" value="${xacro.load_yaml('$(find prius_vehicle_description)/config/vehicle_info.param.yaml')}"/>
+  <!-- <xacro:property name="vehicle_info" value="${xacro.load_yaml('$(find prius_vehicle_description)/config/vehicle_info.param.yaml')}"/> -->
   <!-- vehicle body -->
-  <link name="base_link">
-    <visual>
-      <origin xyz="${vehicle_info['/**']['ros__parameters']['wheel_base']/2.0} 0 0" rpy="${pi/2.0} 0 ${pi}"/>
-      <geometry>
-        <mesh filename="package://prius_vehicle_description/mesh/lexus.dae" scale="1 1 1"/>
-      </geometry>
-    </visual>
-  </link>
+  <!-- <link name="base_link"> -->
+  <!--   <visual> -->
+  <!--     <origin xyz="${vehicle_info['/**']['ros__parameters']['wheel_base']/2.0} 0 0" rpy="${pi/2.0} 0 ${pi}"/> -->
+  <!--     <geometry> -->
+  <!--       <mesh filename="package://prius_description/models/prius/meshes/Hybrid.obj" scale="1 1 1"/> -->
+  <!--     </geometry> -->
+  <!--   </visual> -->
+  <!-- </link> -->
 </robot>
